Commit message: corrected hw0 robot urdf file

File: hw0/rprbot.urdf (robot description, URDF)
Before this commit: robot rprbot, 4 links, 3 joints
Joints:
- joint j0: origin xyz=0 0 0 rpy=0.523599 0 0 -> xyz=0 0 0 rpy=0 0 0

Commit message: corrected hw0 robot urdf last link mass and length

File: hw0/rprbot.urdf (robot description, URDF)
Before this commit: robot rprbot, 4 links, 3 joints
Links:
- link link2: mass 1 -> 2

Commit message: corrected hw0 robot urdf last link visuals

File: hw0/rprbot.urdf (robot description, URDF)
Before this commit: robot rprbot, 4 links, 3 joints
Links:
- link link2: geometry visual cylinder length=2.5 radius=0.03; visual sphere radius=0.09
