Commit message: First pass on urdf

File: stanbot_example/stanbot.urdf (robot description, URDF)
Before this commit: robot stanbot, 32 links, 12 joints
Links:
- removed link left_hand_rz
- removed link left_hip_rx
- removed link left_shoulder_rz
- removed link right_hand_rz
- removed link right_hip_rz
- removed link right_shoulder_rz
- added link head_rx, mass 1e-10
- added link head_ry, mass 1e-10
- added link hip, mass 3; visual mesh filename=../../../model/stanbot/meshes/visual/hip_ascii.obj
- link chest: geometry visual mesh filename=../../../model/stanbot/meshes/visual/chest_ascii.obj
- link head: geometry visual mesh filename=../../../model/stanbot/meshes/visual/head_ascii.obj
- link left_calf: geometry visual mesh filename=../../../model/stanbot/meshes/visual/calf.obj
- link left_foot: geometry visual mesh filename=../../../model/stanbot/meshes/visual/foot.obj
- link left_hand: geometry visual mesh filename=../../../model/stanbot/meshes/visual/hand_ascii.obj
- link left_lower_arm: geometry visual mesh filename=../../../model/stanbot/meshes/visual/lowerArm_ascii.obj
- link left_thigh: geometry visual mesh filename=../../../model/stanbot/meshes/visual/thigh.obj
- link left_upper_arm: geometry visual mesh filename=../../../model/stanbot/meshes/visual/upperArm_ascii.obj
- link right_calf: geometry visual mesh filename=../../../model/stanbot/meshes/visual/calf.obj
- link right_hand: geometry visual mesh filename=../../../model/stanbot/meshes/visual/hand_ascii.obj
- link right_lower_arm: geometry visual mesh filename=../../../model/stanbot/meshes/visual/lowerArm_ascii.obj
- link right_thigh: geometry visual mesh filename=../../../model/stanbot/meshes/visual/thigh.obj
- link right_upper_arm: geometry visual mesh filename=../../../model/stanbot/meshes/visual/upperArm_ascii.obj
Joints:
- removed joint joint1
- removed joint joint10
- removed joint joint11
- removed joint joint12
- removed joint joint2
- removed joint joint3
- removed joint joint4
- removed joint joint5
- removed joint joint6
- removed joint joint7
- removed joint joint8
- removed joint joint9
- added joint j1: type revolute, parent right_foot, child right_calf, origin xyz=0 0.03 0 rpy=0 0 0, axis 1 0 0, limit lower=-2.8973 upper=2.8973 effort=87 velocity=2.1750
- added joint j10: type revolute, parent left_calf, child left_foot, origin xyz=0 0 -0.42 rpy=0 0 0, axis 1 0 0, limit lower=-0.0175 upper=3.7525 effort=12 velocity=2.6100
- added joint j11: type revolute, parent hip, child chest, origin xyz=0 0 0.2 rpy=0 0 0, axis 1 0 0, limit lower=-0.0175 upper=3.7525 effort=12 velocity=2.6100
- added joint j12: type revolute, parent chest, child right_shoulder_rx, origin xyz=0 0 0 rpy=0.5 0.5 0.2, axis 1 0 0, limit lower=-2.8973 upper=2.8973 effort=12 velocity=2.6100
- added joint j13: type revolute, parent right_shoulder_rx, child right_shoulder_ry, origin xyz=0 0 0 rpy=0 0 0, axis 0 1 0, limit lower=-2.8973 upper=2.8973 effort=12 velocity=2.6100
- added joint j14: type revolute, parent right_shoulder_ry, child right_upper_arm, origin xyz=0 0 0 rpy=0 0 0, axis 0 0 1, limit lower=-2.8973 upper=2.8973 effort=12 velocity=2.6100
- added joint j15: type revolute, parent right_upper_arm, child right_lower_arm, origin xyz=0 0 0 rpy=0 0 0, axis 1 0 0, limit lower=-2.8973 upper=2.8973 effort=12 velocity=2.6100
- added joint j16: type revolute, parent right_lower_arm, child right_hand_rx, origin xyz=0 0 0 rpy=0 0 0, axis 1 0 0, limit lower=-2.8973 upper=2.8973 effort=12 velocity=2.6100
- added joint j17: type revolute, parent right_hand_rx, child right_hand_ry, origin xyz=0 0 0 rpy=0 0 0, axis 0 1 0, limit lower=-2.8973 upper=2.8973 effort=12 velocity=2.6100
- added joint j18: type revolute, parent right_hand_ry, child right_hand, origin xyz=0 0 0 rpy=0 0 0, axis 0 0 1, limit lower=-2.8973 upper=2.8973 effort=12 velocity=2.6100
- added joint j19: type revolute, parent chest, child left_shoulder_rx, origin xyz=0 0 0 rpy=0 0 0, axis 1 0 0, limit lower=-2.8973 upper=2.8973 effort=12 velocity=2.6100
- added joint j2: type revolute, parent right_calf, child right_thigh, origin xyz=0 0 0.4 rpy=0 0 0, axis 1 0 0, limit lower=-1.7628 upper=1.7628 effort=87 velocity=2.1750
- added joint j20: type revolute, parent left_shoulder_rx, child left_shoulder_ry, origin xyz=0 0 0 rpy=0 0 0, axis 0 1 0, limit lower=-2.8973 upper=2.8973 effort=12 velocity=2.6100
- added joint j21: type revolute, parent left_shoulder_ry, child left_upper_arm, origin xyz=0 0 0 rpy=0 0 0, axis 0 0 1, limit lower=-2.8973 upper=2.8973 effort=12 velocity=2.6100
- added joint j22: type revolute, parent left_upper_arm, child left_lower_arm, origin xyz=0 0 0 rpy=0 0 0, axis 1 0 0, limit lower=-2.8973 upper=2.8973 effort=12 velocity=2.6100
- added joint j23: type revolute, parent left_lower_arm, child left_hand_rx, origin xyz=0 0 0 rpy=0 0 0, axis 1 0 0, limit lower=-2.8973 upper=2.8973 effort=12 velocity=2.6100
- added joint j24: type revolute, parent left_hand_rx, child left_hand_ry, origin xyz=0 0 0 rpy=0 0 0, axis 0 1 0, limit lower=-2.8973 upper=2.8973 effort=12 velocity=2.6100
- added joint j25: type revolute, parent left_hand_ry, child left_hand, origin xyz=0 0 0 rpy=0 0 0, axis 0 0 1, limit lower=-2.8973 upper=2.8973 effort=12 velocity=2.6100
- added joint j26: type revolute, parent chest, child head_rx, origin xyz=0 0 0 rpy=0 0 0, axis 1 0 0, limit lower=-2.8973 upper=2.8973 effort=12 velocity=2.6100
- added joint j27: type revolute, parent head_rx, child head_ry, origin xyz=0 0 0 rpy=0 0 0, axis 0 1 0, limit lower=-2.8973 upper=2.8973 effort=12 velocity=2.6100
- added joint j28: type revolute, parent head_rx, child head, origin xyz=0 0 0.33 rpy=0 0 0, axis 0 0 1, limit lower=-2.8973 upper=2.8973 effort=12 velocity=2.6100
- added joint j3: type revolute, parent right_thigh, child right_hip_rx, origin xyz=0 0 0 rpy=0 0 0, axis 1 0 0, limit lower=-2.8973 upper=2.8973 effort=87 velocity=2.1750
- added joint j4: type revolute, parent right_hip_rx, child right_hip_ry, origin xyz=0 0 0 rpy=0 0 0, axis 0 1 0, limit lower=-2.8973 upper=2.8973 effort=87 velocity=2.1750
- added joint j5: type revolute, parent right_hip_ry, child hip, origin xyz=0 0 0.4 rpy=0 0 0, axis 0 0 1, limit lower=-2.8973 upper=2.8973 effort=87 velocity=2.1750
- added joint j6: type revolute, parent hip, child left_hip_rz, origin xyz=0.12 0 0 rpy=0 0 0, axis 0 0 1, limit lower=-3.0718 upper=-0.0698 effort=87 velocity=2.1750
- added joint j7: type revolute, parent left_hip_rz, child left_hip_ry, origin xyz=0 0 0 rpy=0 0 0, axis 0 1 0, limit lower=-3.0718 upper=-0.0698 effort=87 velocity=2.1750
- added joint j8: type revolute, parent left_hip_ry, child left_thigh, origin xyz=0 0 0 rpy=0 0 0, axis 1 0 0, limit lower=-3.0718 upper=-0.0698 effort=87 velocity=2.1750
- added joint j9: type revolute, parent left_thigh, child left_calf, origin xyz=0 0 -0.4 rpy=0 0 0, axis 1 0 0, limit lower=-2.8973 upper=2.8973 effort=12 velocity=2.6100

Commit message: Working stanbot demo

File: stanbot_example/stanbot.urdf (robot description, URDF)
Before this commit: robot stanbot, 29 links, 28 joints
Links:
- added link left_foot_rx, mass 1e-10
- added link left_foot_ry, mass 1e-10
- link chest: mass 3 -> 4
- link hip: mass 3 -> 4
- link left_calf: mass 3 -> 4
- link left_foot: mass 2 -> 4
- link left_thigh: mass 3 -> 4
- link right_thigh: mass 3 -> 4
Joints:
- added joint j29: type revolute, parent head_rx, child head_ry, origin xyz=0 0 0 rpy=0 0 0, axis 0 1 0, limit lower=-2.8973 upper=2.8973 effort=12 velocity=2.6100
- added joint j30: type revolute, parent head_ry, child head, origin xyz=0 0 0 rpy=0 0 0, axis 0 0 1, limit lower=-2.8973 upper=2.8973 effort=12 velocity=2.6100
- joint j1: origin xyz=0 0.03 0 rpy=0 0 0 -> xyz=0 0.03 0.02 rpy=0 0 0
- joint j10: child left_foot -> left_foot_rx; origin xyz=0 0 -0.42 rpy=0 0 0 -> xyz=0 0 -0.4 rpy=0 0 0
- joint j11: axis 1 0 0 -> 0 1 0; child chest -> left_foot_ry; origin xyz=0 0 0.2 rpy=0 0 0 -> xyz=0 0 0 rpy=0 0 0; parent hip -> left_foot_rx
- joint j12: axis 1 0 0 -> 0 0 1; child right_shoulder_rx -> left_foot; limit lower=-2.8973 upper=2.8973 effort=12 velocity=2.6100 -> lower=-0.0175 upper=3.7525 effort=12 velocity=2.6100; origin xyz=0 0 0 rpy=0.5 0.5 0.2 -> xyz=0 0 0 rpy=0 0 0; parent chest -> left_foot_ry
- joint j13: axis 0 1 0 -> 1 0 0; child right_shoulder_ry -> chest; limit lower=-2.8973 upper=2.8973 effort=12 velocity=2.6100 -> lower=-0.0175 upper=3.7525 effort=12 velocity=2.6100; origin xyz=0 0 0 rpy=0 0 0 -> xyz=0.06 0 0.2 rpy=0 0 0; parent right_shoulder_rx -> hip
- joint j14: axis 0 0 1 -> 1 0 0; child right_upper_arm -> right_shoulder_rx; origin xyz=0 0 0 rpy=0 0 0 -> xyz=-0.14 0 0.24 rpy=0 0 0; parent right_shoulder_ry -> chest
- joint j15: axis 1 0 0 -> 0 1 0; child right_lower_arm -> right_shoulder_ry; parent right_upper_arm -> right_shoulder_rx
- joint j16: axis 1 0 0 -> 0 0 1; child right_hand_rx -> right_upper_arm; parent right_lower_arm -> right_shoulder_ry
- joint j17: axis 0 1 0 -> 1 0 0; child right_hand_ry -> right_lower_arm; origin xyz=0 0 0 rpy=0 0 0 -> xyz=0 0 -0.3 rpy=0 0 0; parent right_hand_rx -> right_upper_arm
- joint j18: axis 0 0 1 -> 1 0 0; child right_hand -> right_hand_rx; origin xyz=0 0 0 rpy=0 0 0 -> xyz=0 0 -0.3 rpy=0 0 0; parent right_hand_ry -> right_lower_arm
- joint j19: axis 1 0 0 -> 0 1 0; child left_shoulder_rx -> right_hand_ry; parent chest -> right_hand_rx
- joint j20: axis 0 1 0 -> 0 0 1; child left_shoulder_ry -> right_hand; parent left_shoulder_rx -> right_hand_ry
- joint j21: axis 0 0 1 -> 1 0 0; child left_upper_arm -> left_shoulder_rx; origin xyz=0 0 0 rpy=0 0 0 -> xyz=0.14 0 0.24 rpy=0 0 0; parent left_shoulder_ry -> chest
- joint j22: axis 1 0 0 -> 0 1 0; child left_lower_arm -> left_shoulder_ry; parent left_upper_arm -> left_shoulder_rx
- joint j23: axis 1 0 0 -> 0 0 1; child left_hand_rx -> left_upper_arm; parent left_lower_arm -> left_shoulder_ry
- joint j24: axis 0 1 0 -> 1 0 0; child left_hand_ry -> left_lower_arm; origin xyz=0 0 0 rpy=0 0 0 -> xyz=0 0 -0.3 rpy=0 0 0; parent left_hand_rx -> left_upper_arm
- joint j25: axis 0 0 1 -> 1 0 0; child left_hand -> left_hand_rx; origin xyz=0 0 0 rpy=0 0 0 -> xyz=0 0 -0.3 rpy=0 0 0; parent left_hand_ry -> left_lower_arm
- joint j26: axis 1 0 0 -> 0 1 0; child head_rx -> left_hand_ry; parent chest -> left_hand_rx
- joint j27: axis 0 1 0 -> 0 0 1; child head_ry -> left_hand; parent head_rx -> left_hand_ry
- joint j28: axis 0 0 1 -> 1 0 0; child head -> head_rx; origin xyz=0 0 0.33 rpy=0 0 0 -> xyz=0 0 0.30 rpy=0 0 0; parent head_rx -> chest
- joint j3: origin xyz=0 0 0 rpy=0 0 0 -> xyz=0 0 0.4 rpy=0 0 0
- joint j5: origin xyz=0 0 0.4 rpy=0 0 0 -> xyz=0 0 0 rpy=0 0 0
