Commit message: modified panda urdf

File: urdf_models/panda/panda_arm.urdf (robot description, URDF)
Before this commit: robot panda, 9 links, 8 joints
Links:
- removed link end-effector
- link link1: mass 3 -> 4
- link link3: mass 2 -> 3
- link link4: mass 2 -> 3
- link link5: mass 2 -> 3
- link link6: mass 1.5 -> 2
- link link7: mass 1.8 -> 1.0; geometry visual box size=0.15 0.15 0.01; visual mesh filename=meshes/visual/link7.obj
Joints:
- removed joint joint_ee
