Commit message: Scaled bat, simulation and controller working together, bug with redis key?

File: urdf_models/panda/panda_arm_bat.urdf (robot description, URDF)
Before this commit: robot panda_arm_bat, 9 links, 8 joints
Links:
- link end-effector: geometry collision cylinder length=0.5 radius=0.025; visual mesh filename=meshes/visual/Bat.obj scale=0.05 0.05 0.05
Joints:
- joint joint_ee: origin xyz=0.2 0 0.13 rpy=0 1.5708 0 -> xyz=0.4 0 0.13 rpy=0 1.5708 0

Commit message: All new changes plus optitrack stuff

File: urdf_models/panda/panda_arm_bat.urdf (robot description, URDF)
Before this commit: robot panda_arm_bat, 9 links, 8 joints
Links:
- link end-effector: mass 1.0 -> 5.0; geometry collision box size=1.35 .175 0.01; visual box size=1.35 .175 0.01
Joints:
- joint joint_ee: origin xyz=0.4 0 0.13 rpy=0 1.5708 0 -> xyz=0.55 0 0.13 rpy=0 1.5708 0

Commit message: Working batting

File: urdf_models/panda/panda_arm_bat.urdf (robot description, URDF)
Before this commit: robot panda_arm_bat, 9 links, 8 joints
Joints:
- joint joint_ee: origin xyz=0.55 0 0.13 rpy=0 1.5708 0 -> xyz=0.55 0 0.13 rpy=0 1.5708 -0.2

Commit message: Good swinging, new bat mtl, and button + optitrack position working

File: urdf_models/panda/panda_arm_bat.urdf (robot description, URDF)
Before this commit: robot panda_arm_bat, 9 links, 8 joints
Links:
- link end-effector: geometry collision box size=1.2 .175 0.01; visual mesh filename=meshes/visual/Bat.obj scale=0.05 0.05 0.05
Joints:
- joint joint_ee: origin xyz=0.55 0 0.13 rpy=0 1.5708 -0.2 -> xyz=0.55 0 0.15 rpy=0 1.5708 -0.2
