Commit message: Fixed compatibility

File: project_starter/mmp_panda/mmp_panda.urdf (robot description, URDF)
Before this commit: robot mmp_panda, 11 links, 10 joints
Links:
- link base_link: mass 64.6 -> 1

File: project_starter/panda/panda_arm_hand.urdf (robot description, URDF)
Before this commit: robot panda_arm_hand, 10 links, 9 joints
Links:
- link leftfinger: geometry collision box size=0.02 0.01 0.02; visual mesh filename=../../../urdf_models/panda/meshes/visual/finger.obj
- link rightfinger: geometry collision box size=0.02 0.01 0.02; visual mesh filename=../../../urdf_models/panda/meshes/visual/finger.obj
