Commit message: reorganized urdf files

File: urdf_models/mmp_panda/mmp_panda.urdf (robot description, URDF)
Before this commit: robot mmp_panda, 11 links, 10 joints
Links:
- link base_link: geometry visual mesh filename=meshes/panda_BaseCombo.obj
- link link1: geometry visual mesh filename=../panda/meshes/visual/link1.obj
- link link2: geometry visual mesh filename=../panda/meshes/visual/link2.obj
- link link3: geometry visual mesh filename=../panda/meshes/visual/link3.obj
- link link4: geometry visual mesh filename=../panda/meshes/visual/link4.obj
- link link5: geometry visual mesh filename=../panda/meshes/visual/link5.obj
- link link6: geometry visual mesh filename=../panda/meshes/visual/link6.obj
- link link7: geometry visual mesh filename=../panda/meshes/visual/link7.obj

File: urdf_models/mmp_two_arm_panda/mmp_panda_two_arm.urdf (robot description, URDF)
Before this commit: robot mmp_panda, 18 links, 17 joints
Links:
- link base_link: geometry visual mesh filename=meshes/mmp_panda_two_arm_base.obj
- link link1_left: geometry visual mesh filename=../panda/meshes/visual/link1.obj
- link link1_right: geometry visual mesh filename=../panda/meshes/visual/link1.obj
- link link2_left: geometry visual mesh filename=../panda/meshes/visual/link2.obj
- link link2_right: geometry visual mesh filename=../panda/meshes/visual/link2.obj
- link link3_left: geometry visual mesh filename=../panda/meshes/visual/link3.obj
- link link3_right: geometry visual mesh filename=../panda/meshes/visual/link3.obj
- link link4_left: geometry visual mesh filename=../panda/meshes/visual/link4.obj
- link link4_right: geometry visual mesh filename=../panda/meshes/visual/link4.obj
- link link5_left: geometry visual mesh filename=../panda/meshes/visual/link5.obj
- link link5_right: geometry visual mesh filename=../panda/meshes/visual/link5.obj
- link link6_left: geometry visual mesh filename=../panda/meshes/visual/link6.obj
- link link6_right: geometry visual mesh filename=../panda/meshes/visual/link6.obj
- link link7_left: geometry visual mesh filename=../panda/meshes/visual/link7.obj
- link link7_right: geometry visual mesh filename=../panda/meshes/visual/link7.obj

File: urdf_models/ocean1/Divebot_Hybrid.urdf (robot description, URDF)
Before this commit: robot Divebot, 21 links, 20 joints
Links:
- link Body: geometry visual mesh filename=ocean1_graphics/O2_body_new_head.obj scale=0.85 0.85 0.85
- link elbow_left: geometry visual mesh filename=ocean1_graphics/elbow_left.obj
- link elbow_right: geometry visual mesh filename=ocean1_graphics/elbow_right.obj
- link endEffector_left: geometry visual mesh filename=ocean1_graphics/HandO2_small.obj
- link endEffector_right: geometry visual mesh filename=ocean1_graphics/HandO2_small.obj
- link lowerArm_left: geometry visual mesh filename=ocean1_graphics/lowerArm_left.obj
- link lowerArm_right: geometry visual mesh filename=ocean1_graphics/lowerArm_right.obj
- link shoulderL_left: geometry visual mesh filename=ocean1_graphics/shoulderL_left.obj
- link shoulderL_right: geometry visual mesh filename=ocean1_graphics/shoulderL_right.obj
- link shoulderT_left: geometry visual mesh filename=ocean1_graphics/shoulderT_left.obj
- link shoulderT_right: geometry visual mesh filename=ocean1_graphics/shoulderT_right.obj
- link upperArm_left: geometry visual mesh filename=ocean1_graphics/upperArm_left.obj
- link upperArm_right: geometry visual mesh filename=ocean1_graphics/upperArm_right.obj
- link wristDiff_left: geometry visual mesh filename=ocean1_graphics/wristDiff_left.obj
- link wristDiff_right: geometry visual mesh filename=ocean1_graphics/wristDiff_right.obj

File: urdf_models/panda/panda_arm_hand.urdf (robot description, URDF)
Before this commit: robot panda_hand, 10 links, 9 joints
Links:
- link leftfinger: geometry collision box size=0.02 0.01 0.02; visual mesh filename=meshes/visual/finger.obj
- link link0: geometry visual mesh filename=meshes/visual/link0.obj
- link link1: geometry visual mesh filename=meshes/visual/link1.obj
- link link2: geometry visual mesh filename=meshes/visual/link2.obj
- link link3: geometry visual mesh filename=meshes/visual/link3.obj
- link link4: geometry visual mesh filename=meshes/visual/link4.obj
- link link5: geometry visual mesh filename=meshes/visual/link5.obj
- link link6: geometry visual mesh filename=meshes/visual/link6.obj
- link link7: geometry visual mesh filename=meshes/visual/hand.obj; visual mesh filename=meshes/visual/link7.obj
- link rightfinger: geometry collision box size=0.02 0.01 0.02; visual mesh filename=meshes/visual/finger.obj
Joints:
- joint finger_joint2: limit lower=0.0 upper=0.04 effort=20 velocity=0.2 -> lower=-0.04 upper=0 effort=20 velocity=0.2

File: urdf_models/toro/toro.urdf (robot description, URDF)
Before this commit: robot DLR_TORO, 34 links, 33 joints
Links:
- added link LL_end_effector, mass 0.001; collision box size=0.2 0.1 0.02
- added link RL_end_effector, mass 0.001; collision box size=0.2 0.1 0.02
- added link la_end_effector, mass 0.1; collision box size=0.1 0.1 0.01; visual box size=0.1 0.1 0.01
- added link ra_end_effector, mass 0.1; collision box size=0.1 0.1 0.01; visual box size=0.1 0.1 0.01
- link LL_KOSY_L1: mass 2.7752200000 -> 3.1576128000; geometry visual mesh filename=meshes/obj/left_lower_hip.stl.obj
- link LL_KOSY_L23: mass 2.2450500000 -> 2.6274499000; geometry visual mesh filename=meshes/obj/kuka-link2.stl.obj
- link LL_KOSY_L4: mass 2.6274500000 -> 2.6220074000; geometry visual mesh filename=meshes/obj/kuka-link3.stl.obj
- link LL_KOSY_L56: mass 5.7035400000 -> 5.7433829000; geometry visual mesh filename=meshes/obj/left_calf.stl.obj
- link LL_ankle: geometry visual mesh filename=meshes/obj/ankle.stl.obj
- link LL_foot: geometry visual mesh filename=meshes/obj/foot.stl.obj
- link RL_KOSY_L1: mass 2.7752200000 -> 3.1576128000; geometry visual mesh filename=meshes/obj/right_lower_hip.stl.obj
- link RL_KOSY_L23: mass 2.2450500000 -> 2.6274499000; geometry visual mesh filename=meshes/obj/kuka-link2.stl.obj
- link RL_KOSY_L4: mass 2.6274500000 -> 2.6220074000; geometry visual mesh filename=meshes/obj/kuka-link3.stl.obj
- link RL_KOSY_L56: mass 5.7035400000 -> 5.7433829000; geometry visual mesh filename=meshes/obj/right_calf.stl.obj
- link RL_ankle: geometry visual mesh filename=meshes/obj/ankle.stl.obj
- link RL_foot: geometry visual mesh filename=meshes/obj/foot.stl.obj
- link floating_virtual1: mass 0.001 -> 1e-9
- link floating_virtual2: mass 0.001 -> 1e-9
- link floating_virtual3: mass 0.001 -> 1e-9
- link floating_virtual4: mass 0.001 -> 1e-9
- link floating_virtual5: mass 0.001 -> 1e-9
- link hip_base: geometry visual mesh filename=meshes/obj/upper_hip.stl.obj
- link la_link1: mass 2.2396100000 -> 2.6220074000; geometry visual mesh filename=meshes/obj/kuka-link1.stl.obj
- link la_link2: mass 1.0993800000 -> 1.0979371000; geometry visual mesh filename=meshes/obj/va_left_shoulder_front.stl.obj
- link la_link3: mass 2.3629100000 -> 2.3628586000; geometry visual mesh filename=meshes/obj/va_left_upper_arm.stl.obj
- link la_link4: mass 0.7187000000 -> 0.7247867400; geometry visual mesh filename=meshes/obj/va_left_lower_elbow.stl.obj
- link la_link5: mass 2.2786200000 -> 2.2114157000; geometry visual mesh filename=meshes/obj/va_left_lower_arm.stl.obj; visual mesh filename=meshes/obj/wrist_cap.stl.obj
- link la_link6: geometry visual mesh filename=meshes/obj/wrist.stl.obj
- link neck_link1: mass 0.3364400000 -> 0.2300000000; geometry visual mesh filename=meshes/obj/neck.stl.obj
- link neck_link2: mass 2.4522900000 -> 1.4522900000; geometry visual mesh filename=meshes/obj/head.stl.obj
- link ra_link1: mass 2.2396100000 -> 2.6220074000; geometry visual mesh filename=meshes/obj/kuka-link1.stl.obj
- link ra_link2: mass 1.0993800000 -> 1.0979371000; geometry visual mesh filename=meshes/obj/va_right_shoulder_front.stl.obj
- link ra_link3: mass 2.3629100000 -> 2.3628586000; geometry visual mesh filename=meshes/obj/va_right_upper_arm.stl.obj
- link ra_link4: mass 0.7187000000 -> 0.7247867400; geometry visual mesh filename=meshes/obj/va_right_lower_elbow.stl.obj
- link ra_link5: mass 2.2786200000 -> 2.2114157000; geometry visual mesh filename=meshes/obj/va_right_lower_arm.stl.obj; visual mesh filename=meshes/obj/wrist_cap.stl.obj
- link ra_link6: geometry visual mesh filename=meshes/obj/wrist.stl.obj
- link trunk: mass 18.9794300000 -> 19.6443820000; geometry visual mesh filename=meshes/obj/trunk.stl.obj
Joints:
- removed joint j1
- removed joint j10
- removed joint j11
- removed joint j12
- removed joint j13
- removed joint j14
- removed joint j15
- removed joint j16
- removed joint j17
- removed joint j18
- removed joint j19
- removed joint j2
- removed joint j20
- removed joint j21
- removed joint j22
- removed joint j23
- removed joint j24
- removed joint j25
- removed joint j26
- removed joint j27
- removed joint j3
- removed joint j4
- removed joint j5
- removed joint j6
- removed joint j7
- removed joint j8
- removed joint j9
- added joint j_la_elbow: type revolute, parent la_link3, child la_link4, origin xyz=0.0300000000 -0.3128000000 -0.0000000000 rpy=0.0000000000 0.0000000000 0.0000000000, axis 0 0 1, limit lower=0 upper=2.5831 effort=40 velocity=2.0944
- added joint j_la_frontal: type revolute, parent la_link1, child la_link2, origin xyz=0.0539500000 0.0000000000 0.0000000000 rpy=-0.5235987756  0.0000000000  0.0000000000, axis 1 0 0, limit lower=-0.2618 upper=3.1416 effort=100 velocity=2.7402
- added joint j_la_sagittal: type revolute, parent trunk, child la_link1, origin xyz=0.0000000000 0.2590563550 0.3552250220 rpy=2.0943951024 0.0000000000 0.0000000000, axis 0 0 1, limit lower=-2.0944 upper=2.0944 effort=100 velocity=2.7402
- added joint j_la_self_rotation: type revolute, parent la_link2, child la_link3, axis 0 1 0, limit lower=-1.8326 upper=1.8326 effort=40 velocity=2.0944
- added joint j_la_wrist_frontal: type revolute, parent la_link5, child la_link6, origin xyz=0.0140000000 -0.0000000000 -0.0000000000 rpy=0.0000000000 0.0000000000 0.0000000000, axis 1 0 0, limit lower=-1.8326 upper=1.8326 effort=40 velocity=2.0944
- added joint j_la_wrist_self_rotation: type revolute, parent la_link4, child la_link5, origin xyz=-0.0300000000 -0.3058000000  0.0115000000 rpy=0.0000000000 0.0000000000 0.0000000000, axis 0 1 0, limit lower=-2.5307 upper=2.0595 effort=40 velocity=2.0944
- added joint j_lfoot_fixed: type fixed, parent LL_foot, child LL_end_effector, origin xyz=0.04 0 -0.08 rpy=0 0 0
- added joint j_lhand_fixed: type fixed, parent la_link6, child la_end_effector, origin xyz=0 -0.056 0 rpy=-1.5707963268  0.0000000000 0.0000000000
- added joint j_ll_ankle_frontal: type revolute, parent LL_KOSY_L56, child LL_ankle, origin xyz=0.0000000000 -0.0220500000 -0.4000000000 rpy=0 0 0, axis 1 0 0, limit lower=-0.3403 upper=0.3403 effort=50 velocity=2.0944
- added joint j_ll_ankle_sagittal: type revolute, parent LL_ankle, child LL_foot, origin xyz=-0.0000000000 0.0000000000 -0.0200000 rpy=0 0 0, axis 0 1 0, limit lower=-0.7854 upper=0.7854 effort=165 velocity=3.0718
- added joint j_ll_frontal: type revolute, parent hip_base, child LL_KOSY_L1, origin xyz=0.0000000000 0.1000000000 -0.1254789680 rpy=0 0 0, axis  1 0 0 , limit lower=-0.7804 upper=1.5708 effort=176 velocity=1.9199
- added joint j_ll_knee: type revolute, parent LL_KOSY_L4, child LL_KOSY_L56, origin xyz=0.0000000000 0.0000000000 -0.3999000880 rpy=0 0 0, axis 0 1 0, limit lower=-1.8326 upper=1.8326 effort=165 velocity=3.0718
- added joint j_ll_sagittal: type revolute, parent LL_KOSY_L1, child LL_KOSY_L23, origin xyz=0.0000000000 0.0350000000 -0.1200000000 rpy=0 0 0, axis 0 1 0, limit lower=-2.0071 upper=1.5708 effort=100 velocity=2.7402
- added joint j_ll_self_rotation: type revolute, parent LL_KOSY_L23, child LL_KOSY_L4, axis 0 0 1, limit lower=-2.0944 upper=2.0944 effort=100 velocity=2.7402
- added joint j_neck_sagittal: type revolute, parent neck_link1, child neck_link2, origin xyz=-0.035 0 0.05, axis 0 1 0, limit lower=-0.5236 upper=1.5708 effort=8.4 velocity=4.7124
- added joint j_neck_self_rotation: type revolute, parent trunk, child neck_link1, origin xyz=0.0548813000 0.0000000000 0.3505590000 rpy=0 0 0, axis 0 0 1, limit lower=-1.5708 upper=1.5708 effort=8.4 velocity=4.7124
- added joint j_ra_elbow: type revolute, parent ra_link3, child ra_link4, origin xyz=-0.0000000000 -0.0300000000  0.3129000000 rpy=0.0000000000 0.0000000000 0.0000000000, axis 1 0 0, limit lower=0 upper=2.5831 effort=40 velocity=2.0944
- added joint j_ra_frontal: type revolute, parent ra_link1, child ra_link2, origin xyz=0.0539500000 0.0000000000 0.0000000000 rpy=0.0000000000 0.0000000000 1.5707963268, axis 0 1 0, limit lower=-0.2618 upper=3.1416 effort=100 velocity=2.7402
- added joint j_ra_sagittal: type revolute, parent trunk, child ra_link1, origin xyz=0.0000000000 -0.2590563550  0.3552250220 rpy=1.0471975512 0.0000000000 0.0000000000, axis 0 0 1, limit lower=-2.0944 upper=2.0944 effort=100 velocity=2.7402
- added joint j_ra_self_rotation: type revolute, parent ra_link2, child ra_link3, origin xyz=0.0000000000 0.0000000000 0.0000000000 rpy=-3.1415926536 -1.0471975512 -3.1415926536, axis 0 0 1, limit lower=-1.8326 upper=1.8326 effort=40 velocity=2.0944
- added joint j_ra_wrist_frontal: type revolute, parent ra_link5, child ra_link6, origin xyz=-0.0000000000 -0.0140000000  0.00000000 rpy=0.0000000000 0.0000000000 0.0000000000, axis 0 1 0, limit lower=-1.8326 upper=1.8326 effort=35 velocity=2.0944
- added joint j_ra_wrist_self_rotation: type revolute, parent ra_link4, child ra_link5, origin xyz=-0.0115000000  0.0300000000  0.3059000000 rpy=0.0000000000 0.0000000000 0.0000000000, axis 0 0 1, limit lower=-2.5307 upper=2.0595 effort=40 velocity=2.0944
- added joint j_rfoot_fixed: type fixed, parent RL_foot, child RL_end_effector, origin xyz=0.04 0 -0.08 rpy=0 0 0
- added joint j_rhand_fixed: type fixed, parent ra_link6, child ra_end_effector, origin xyz=0 0 0.056 rpy=-3.1415926536  0.0000000000 -1.5707963268
- added joint j_rl_ankle_frontal: type revolute, parent RL_KOSY_L56, child RL_ankle, origin xyz=-0.0000000000 0.0220500000 -0.4000000000 rpy=0 0 0, axis 1 0 0, limit lower=-0.3403 upper=0.3403 effort=50 velocity=2.0944
- added joint j_rl_ankle_sagittal: type revolute, parent RL_ankle, child RL_foot, origin xyz=-0.0000000000 0.0000000000 -0.0200000 rpy=0 0 0, axis 0 1 0, limit lower=-0.7804 upper=0.7804 effort=165 velocity=3.0718
- added joint j_rl_frontal: type revolute, parent hip_base, child RL_KOSY_L1, origin xyz=-0.0000000000 -0.1000000000 -0.1254789680 rpy=0 0 0, axis 1 0 0, limit lower=-1.5708 upper=0.7854 effort=176 velocity=1.9199
- added joint j_rl_knee: type revolute, parent RL_KOSY_L4, child RL_KOSY_L56, origin xyz=0.0000000000 0.0000000000 -0.3999000880 rpy=0 0 0, axis 0 1 0, limit lower=-1.8326 upper=1.8326 effort=165 velocity=3.0718
- added joint j_rl_sagittal: type revolute, parent RL_KOSY_L1, child RL_KOSY_L23, origin xyz=-0.0000000000 -0.0350000000 -0.1200000000 rpy=0 0 0, axis 0 1 0, limit lower=-2.0071 upper=1.5708 effort=100 velocity=2.7402
- added joint j_rl_self_rotation: type revolute, parent RL_KOSY_L23, child RL_KOSY_L4, axis 0 0 1, limit lower=-2.0944 upper=2.0944 effort=100 velocity=2.7402
- added joint j_waist: type revolute, parent hip_base, child trunk, axis 0 0 1, limit lower=-2.0944 upper=2.0944 effort=100 velocity=2.7402
- joint floating_base_p1: limit lower=5.00 upper=5.00 effort=4000 velocity=1000 -> lower=-500.00 upper=500.00 effort=4000 velocity=1000; origin xyz=0.000000 0.000000 0.00000 rpy=0.000000 0.000000 0.000000 -> xyz=0.000000 0.000000 2.089000 rpy=0.000000 0.000000 0.000000
- joint floating_base_p2: limit lower=5.00 upper=5.00 effort=4000 velocity=1000 -> lower=-500.00 upper=500.00 effort=4000 velocity=1000
- joint floating_base_p3: limit lower=5.00 upper=5.00 effort=4000 velocity=1000 -> lower=-500.00 upper=500.00 effort=4000 velocity=1000
- joint floating_base_r1: limit lower=50.00 upper=5.00 effort=4000 velocity=1000 -> lower=-500.00 upper=500.00 effort=4000 velocity=1000
- joint floating_base_r2: axis 0 1 0 -> 0 0 1; limit lower=50.00 upper=5.00 effort=4000 velocity=1000 -> lower=-500.00 upper=500.00 effort=4000 velocity=1000
- joint floating_base_r3: axis 0 0 1 -> 0 1 0; limit lower=50.00 upper=5.00 effort=4000 velocity=1000 -> lower=-500.00 upper=500.00 effort=4000 velocity=1000
