Commit message: Added spot example

File: project_starter/toro/toro.urdf (robot description, URDF)
Before this commit: robot DLR_TORO, 38 links, 37 joints
Joints:
- removed joint j_lhand_fixed
- removed joint j_rhand_fixed
- added joint j_lhand_revolute: type revolute, parent la_link6, child la_end_effector, origin xyz=0 -0.056 0 rpy=-1.5707963268  0.0000000000 0.0000000000, axis 0 0 1, limit lower=-1.8326 upper=1.8326 effort=35 velocity=2.0944
- added joint j_rhand_revolute: type revolute, parent ra_link6, child ra_end_effector, origin xyz=0 0 0.056 rpy=-3.1415926536  0.0000000000 -1.5707963268, axis 0 0 1, limit lower=-1.8326 upper=1.8326 effort=35 velocity=2.0944
- joint j_la_elbow: limit lower=0 upper=2.5831 effort=40 velocity=2.0944 -> lower=0.5 upper=2.5831 effort=40 velocity=2.0944
- joint j_ll_knee: limit lower=-1.8326 upper=1.8326 effort=165 velocity=3.0718 -> lower=0.2 upper=1.8326 effort=165 velocity=3.0718
- joint j_ra_elbow: limit lower=0 upper=2.5831 effort=40 velocity=2.0944 -> lower=0.5 upper=2.5831 effort=40 velocity=2.0944
- joint j_rl_knee: limit lower=-1.8326 upper=1.8326 effort=165 velocity=3.0718 -> lower=0.2 upper=1.8326 effort=165 velocity=3.0718
