Commit message: added ocean1 example

File: urdf_models/ocean1/ocean1.urdf (robot description, URDF)
Before this commit: robot Divebot, 21 links, 20 joints
Joints:
- joint PrisX_Joint: limit effort=100.0 velocity=3.0 -> lower=-500.00 upper=500.00 effort=4000 velocity=1000
- joint PrisY_Joint: limit effort=100.0 velocity=3.0 -> lower=-500.00 upper=500.00 effort=4000 velocity=1000
- joint PrisZ_Joint: limit effort=100.0 velocity=3.0 -> lower=-500.00 upper=500.00 effort=4000 velocity=1000
- joint RotX_Joint: limit effort=100.0 velocity=3.0 -> lower=-500.00 upper=500.00 effort=4000 velocity=1000
- joint RotY_Joint: limit effort=100.0 velocity=3.0 -> lower=-500.00 upper=500.00 effort=4000 velocity=1000
- joint RotZ_Joint: limit effort=100.0 velocity=3.0 -> lower=-500.00 upper=500.00 effort=4000 velocity=1000
- joint elbow_left_Joint: limit effort=100.0 velocity=3.0 -> lower=-500.00 upper=500.00 effort=4000 velocity=1000
- joint elbow_right_Joint: limit effort=100.0 velocity=3.0 -> lower=-500.00 upper=500.00 effort=4000 velocity=1000
- joint endEffector_left_Joint: limit effort=100.0 velocity=3.0 -> lower=-500.00 upper=500.00 effort=4000 velocity=1000
- joint endEffector_right_Joint: limit effort=100.0 velocity=3.0 -> lower=-500.00 upper=500.00 effort=4000 velocity=1000
- joint lowerArm_left_Joint: limit effort=100.0 velocity=3.0 -> lower=-500.00 upper=500.00 effort=4000 velocity=1000
- joint lowerArm_right_Joint: limit effort=100.0 velocity=3.0 -> lower=-500.00 upper=500.00 effort=4000 velocity=1000
- joint shoulderL_left_Joint: limit effort=100.0 velocity=3.0 -> lower=-500.00 upper=500.00 effort=4000 velocity=1000
- joint shoulderL_right_Joint: limit effort=100.0 velocity=3.0 -> lower=-500.00 upper=500.00 effort=4000 velocity=1000
- joint shoulderT_left_Joint: limit effort=100.0 velocity=3.0 -> lower=-500.00 upper=500.00 effort=4000 velocity=1000
- joint shoulderT_right_Joint: limit effort=100.0 velocity=3.0 -> lower=-500.00 upper=500.00 effort=4000 velocity=1000
- joint upperArm_left_Joint: limit effort=100.0 velocity=3.0 -> lower=-500.00 upper=500.00 effort=4000 velocity=1000
- joint upperArm_right_Joint: limit effort=100.0 velocity=3.0 -> lower=-500.00 upper=500.00 effort=4000 velocity=1000
- joint wristDiff_left_Joint: limit effort=100.0 velocity=3.0 -> lower=-500.00 upper=500.00 effort=4000 velocity=1000
- joint wristDiff_right_Joint: limit effort=100.0 velocity=3.0 -> lower=-500.00 upper=500.00 effort=4000 velocity=1000
