Commit message: Fixed the Flexiv visuals link offset

File: urdf_models/flexiv/flexiv.urdf (robot description, URDF)
Before this commit: robot 4S-Titania, 9 links, 8 joints
Joints:
- joint joint7: origin xyz=-0.055 0.07 0.11 rpy=0.0 -1.5707963478683205 0.0 -> xyz=-0.015 0.07 0.11 rpy=0.0 -1.5707963478683205 0.0
